File: hw_pcb/mbadge25_v2/mbadge25.kicad_sch (KiCad schematic)
At the start: 46 parts, among them J1 USB4105-GF-A, J10 Conn_IO20.RX, J11 Conn_IO19.USBP, J12 Conn_IO18.USBN, J15 Conn_IO4, J16 Conn_IO5, J2 BAT, J20 Conn_IO10, J21 Conn_IO00, J22 Conn_IO01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

Commit message: Cleaned up PR as per review comments
Parts:
- C1, C2: Manufacturer Part Number (none) -> CC1206JKNPOCBN470
- C3, C7: Manufacturer Part Number (none) -> CC1206KRX7R9BB104
- C4, C5, C6: Manufacturer Part Number (none) -> CC1206KKX7R0BB225
- C8, C9: Manufacturer Part Number (none) -> CC1206KKX7R0BB105
- D1: value MSK4005 -> B0520LW-7-F; footprint Library_FP_mbadge25:D_SOD-523 -> Library_FP_mbadge25:D_SOD-123; Manufacturer Part Number (none) -> B0520LW-7-F
- J1: Manufacturer Part Number (none) -> USB4105-GF-A
- R1, R2: Manufacturer Part Number (none) -> RC1206FR-075K1L
- R10, R11, R6, R9: Manufacturer Part Number (none) -> RC1206FR-0710KL
- R3, R4: Manufacturer Part Number (none) -> RC1206FR-0727RL
- R5: Manufacturer Part Number (none) -> RC1206FR-07100KL
- R8: Manufacturer Part Number (none) -> RE1206FRE07220RL
- S1, S2: Manufacturer Part Number (none) -> TC-6601-5.0-160
- T1: value LP0404N3T5G -> SI2303CDS-T1-GE3; Manufacturer Part Number (none) -> SI2303CDS-T1-GE3
- U2: value XC6220B331MR -> AP7366-33W5-7
